Commit message: fix transformations

File: urdf/frame/dji_m100_frame.xacro (robot description, xacro)
@@ -9,6 +9,5 @@
   <!-- The xacro macro xacro:drone_base contains: frame -->
   <xacro:macro name="dji_m100_frame" params="name">
-    <!-- dummy frame to the bottom of the drone -->
-    <link name="${name}_footprint">
+    <link name="${name}_link">
       <inertial>
         <mass value="${base_mass}" />
@@ -22,9 +21,9 @@
       </inertial>
       <visual>
-        <origin xyz="0.35 0.25 -0.14" rpy="${M_PI/2} 0 ${-M_PI/2}" />
+        <origin xyz="-0.35 -0.25 -0.14" rpy="${M_PI/2} 0 ${M_PI/2}" />
         <geometry>
           <mesh filename="package://airsim_img_publisher/meshes/DJI_M100_CAD.STL" scale="0.001 0.001 0.001"/>
         </geometry>
-        <material name="Grey" />
+        <material name="Black" />
       </visual>
       <collision>
@@ -35,12 +34,4 @@
       </collision>
     </link>
-    <!-- base_link frame -->
-    <!-- front center camera (cameraID = 0) -->
-    <link name="${name}_link" />
-    <joint name="${name}_dummy_joint" type="fixed">
-      <parent link="${name}_footprint" />
-      <child link="${name}_link" />
-      <origin xyz="0 0 0" rpy="0 0 ${M_PI}" />
-    </joint>
   </xacro:macro>
 </robot>

File: urdf/robot/dji_m100_airsim.urdf (robot description, URDF)
Before this commit: robot dji_m100_airsim, 7 links, 6 joints
Links:
- removed link base_footprint
- link base_link: mass None -> 2.432; geometry collision cylinder length=0.218 radius=0.498; visual mesh filename=package://airsim_img_publisher/meshes/DJI_M100_CAD.STL scale=0.001 0.001 0.001
Joints:
- removed joint base_dummy_joint
- joint bottom_back_cam: origin xyz=-0.046 0 0 rpy=0 1.57079632679 0 -> xyz=-0.046 0 0 rpy=3.14159265359 0 -1.57079632679
- joint bottom_center_cam: origin xyz=0 0 -0.012 rpy=0 1.57079632679 0 -> xyz=0 0 -0.012 rpy=3.14159265359 0 -1.57079632679
- joint front_center_cam: origin xyz=0.046 0 0 rpy=0 1.57079632679 0 -> xyz=0.046 0 0 rpy=3.14159265359 0 -1.57079632679
- joint front_left_cam: origin xyz=0.046 -0.0125 0 rpy=0 1.57079632679 0 -> xyz=0.046 -0.0125 0 rpy=3.14159265359 0 -1.57079632679
- joint front_right_cam: origin xyz=0.046 0.0125 0 rpy=0 1.57079632679 0 -> xyz=0.046 0.0125 0 rpy=3.14159265359 0 -1.57079632679

File: urdf/sensors/airsim_cam.xacro (robot description, xacro)
@@ -9,5 +9,5 @@
       <parent link="${name}_link" />
       <child link="front_center_optical" />
-      <origin xyz="0.046 0 0" rpy="0 ${M_PI/2} 0" />
+      <origin xyz="0.046 0 0" rpy="${M_PI} 0 -${M_PI/2}" />
     </joint>
     <!-- front left camera (cameraID = 1) -->
@@ -16,5 +16,5 @@
       <parent link="${name}_link" />
       <child link="front_left_optical" />
-      <origin xyz="0.046 -0.0125 0" rpy="0 ${M_PI/2} 0" />
+      <origin xyz="0.046 -0.0125 0" rpy="${M_PI} 0 -${M_PI/2}" />
     </joint>
     <!-- front right camera (cameraID = 2) -->
@@ -23,5 +23,5 @@
       <parent link="${name}_link" />
       <child link="front_right_optical" />
-      <origin xyz="0.046 0.0125 0" rpy="0 ${M_PI/2} 0" />
+      <origin xyz="0.046 0.0125 0" rpy="${M_PI} 0 -${M_PI/2}" />
     </joint>
     <!-- bottom center camera (cameraID = 3) -->
@@ -30,5 +30,5 @@
       <parent link="${name}_link" />
       <child link="bottom_center_optical" />
-      <origin xyz="0 0 -0.012" rpy="0 ${M_PI/2} 0" />
+      <origin xyz="0 0 -0.012" rpy="${M_PI} 0 -${M_PI/2}" />
     </joint>
     <!-- bottom back camera (cameraID = 4) -->
@@ -37,5 +37,5 @@
       <parent link="${name}_link" />
       <child link="bottom_back_optical" />
-      <origin xyz="-0.046 0 0" rpy="0 ${M_PI/2} 0" />
+      <origin xyz="-0.046 0 0" rpy="${M_PI} 0 -${M_PI/2}" />
     </joint>
   </xacro:macro>
